File: lab-5.kicad_sch (KiCad schematic)
At the start: 48 parts, among them J2 USB_C_Receptacle, J6 Conn_01x24_Pin, SW1 NRST, SW2 BOOT, SW3 USER, U1 LM66100DCK, U2 LM66100DCK, U3 STM32F405RGTx, U5 AP2112K-3.3, Y1 8 MHz

Commit message: add BMP280 via I2C
Parts:
- added C10, C9: 100n, Capacitor_SMD:C_0402_1005Metric, symbol Device:C
- added U4: BMP280, Package_LGA:Bosch_LGA-8_2x2.5mm_P0.65mm_ClockwisePinNumbering, symbol Sensor_Pressure:BMP280
- added U6: BMI160, Package_LGA:Bosch_LGA-14_3x2.5mm_P0.5mm, symbol Sensor_Motion:BMI160
- added U7: BMM150, Package_CSP:WLCSP-12_1.56x1.56mm_P0.4mm, symbol Sensor_Magnetic:BMM150
Connections:
- net +3.3V: now also C10.1, C9.2, U4.2 (CSB), U4.6 (VDDIO), U4.8 (VDD)
- net GND: now also C10.2, C9.1, U4.1 (GND), U4.5 (SDO), U4.7 (GND)
- net I2C1_SCL: now also U4.4 (SCK); no longer J6.5 (Pin_5)
- net I2C1_SDA: now also U4.3 (SDI); no longer J6.4 (Pin_4)
- new net: U7.C5 (GND), U7.E1 (GND), U7.E3 (GND)
- no-connect marks 0 -> 2
Other:
- moved on the sheet: R11, R12, R14

Commit message: added the BMI160 and logo, full board refactoring
Signed-off-by: Yehor Bilous <bilous801@gmail.com>
Parts:
- removed J6: Conn_01x24_Pin, Connector_PinHeader_2.54mm:PinHeader_1x24_P2.54mm_Vertical, symbol Connector:Conn_01x24_Pin
- removed R14: 4.7k, Resistor_SMD:R_0402_1005Metric, symbol Device:R
- added C17, C18: 100n, Capacitor_SMD:C_0402_1005Metric, symbol Device:C
- added J1: Conn_01x04_Pin, Connector_PinHeader_2.54mm:PinHeader_1x04_P2.54mm_Vertical, symbol Connector:Conn_01x04_Pin
- added J3, J4: Conn_01x15_Pin, Connector_PinHeader_2.54mm:PinHeader_1x15_P2.54mm_Vertical, symbol Connector:Conn_01x15_Pin
Connections:
- net +3.3V: now also U6.5 (VDDIO), U6.8 (VDD), C17.1, C18.1
- net +3.3V_STLINK_IN: now also J1.3 (Pin_3)
- net GND: now also U6.6 (GNDIO), U6.7 (GND), C17.2, C18.2, J1.4 (Pin_4)
- net I2C2_SCL: now reaches U7.A3 (SCK)
- net I2C2_SCL: now also U3.29 (PB10)
- net I2C2_SDA: now reaches U7.B4 (SDI)
- net I2C2_SDA: now also U3.30 (PB11)
- net GPIO_EXTI2: now reaches U7.D2 (INT)
- net GPIO_EXTI2: now also U3.28 (PB2)
- net SPI1_NSS: now reaches U3.20 (PA4)
- net SPI1_NSS: now also U6.12 (CSB)
- net SPI1_SCK: now reaches U3.21 (PA5)
- net SPI1_SCK: now also U6.13 (SCx)
- net SPI1_MISO: now reaches U3.22 (PA6)
- net SPI1_MISO: now also U6.1 (SDO)
- net SPI1_MOSI: now reaches U3.23 (PA7)
- net SPI1_MOSI: now also U6.14 (SDx)
- net GPIO_EXTI4: now reaches U3.24 (PC4)
- net GPIO_EXTI4: now also U6.4 (INT1)
- net GPIO_EXTI5: now reaches U3.25 (PC5)
- net GPIO_EXTI5: now also U6.9 (INT2)
- net GPIOC_6: no longer names the net of U3.37 (PC6)
- net GPIOC_7: no longer names the net of U3.38 (PC7)
- net GPIOC_8: no longer names the net of U3.39 (PC8)
- net GPIOC_9: no longer names the net of U3.40 (PC9)
- net SPI_MISO: no longer names the net of U3.35 (PB14)
- net SPI_MOSI: no longer names the net of U3.36 (PB15)
- net SPI_NSS: no longer names the net of U3.33 (PB12)
- net SPI_SCK: no longer names the net of U3.34 (PB13)
- net SWCLK renamed SYS_JTMS_SWCLK
- net SYS_JTMS_SWCLK: now also J1.1 (Pin_1)
- net SWDIO renamed SYS_JTMS_SWDIO
- net SYS_JTMS_SWDIO: now also J1.2 (Pin_2)
- net UART_RX: no longer names the net of U3.52 (PC11)
- net UART_TX: no longer names the net of U3.51 (PC10)
- net USER renamed USER_BUTTON
- no-connect marks 2 -> 4
Other:
- note removed: "Header"
- moved on the sheet: C13, C14, R11, R12, R7, SW3, U7

Commit message: Added bmm150 and connected all other interfaces
Parts:
- added C19, C20: 100n, Capacitor_SMD:C_0402_1005Metric, symbol Device:C
- added R13, R14, R15, R16: 4.7k, Resistor_SMD:R_0402_1005Metric, symbol Device:R
Connections:
- net +3.3V: now also J3.1 (Pin_1), J4.1 (Pin_1), U7.A1 (PS), U7.A5 (CSB), U7.B2 (VDDIO), U7.C1 (SDO), U7.E5 (VDD), C19.2, C20.1, R13.2, R14.1, R15.2, R16.1
- net GND: now also J3.13 (Pin_13), J3.2 (Pin_2), J3.5 (Pin_5), J3.8 (Pin_8), J4.13 (Pin_13), J4.2 (Pin_2), J4.5 (Pin_5), J4.8 (Pin_8), U7.C5 (GND), U7.E1 (GND), U7.E3 (GND), C19.1, C20.2
- net GPIO_EXTI2: now also U7.D4 (DRDY); no longer U7.D2 (INT)
- net I2C1_SCL: now also U7.A3 (SCK)
- net I2C1_SDA: now also U7.B4 (SDI)
- net I2C2_SCL: now also J3.7 (Pin_7), R13.1; no longer U7.A3 (SCK)
- net I2C2_SDA: now also J3.6 (Pin_6), R14.2; no longer U7.B4 (SDI)
- net SPI2_MISO: now reaches J3.10 (Pin_10)
- net SPI2_MISO: now also U3.35 (PB14)
- net SPI2_SCK: now reaches J3.11 (Pin_11)
- net SPI2_SCK: now also U3.34 (PB13)
- net SPI2_NSS: now reaches J3.12 (Pin_12)
- net SPI2_NSS: now also U3.33 (PB12)
- net UART4_RX: now reaches J3.14 (Pin_14)
- net UART4_RX: now also U3.52 (PC11)
- net UART4_TX: now reaches J3.15 (Pin_15)
- net UART4_TX: now also U3.51 (PC10)
- net GPIOB_9: now reaches J3.3 (Pin_3)
- net GPIOB_9: now also U3.62 (PB9)
- net GPIOB_8: now reaches J3.4 (Pin_4)
- net GPIOB_8: now also U3.61 (PB8)
- net SPI2_MOSI: now reaches J3.9 (Pin_9)
- net SPI2_MOSI: now also U3.36 (PB15)
- net GPIOC_6: now reaches U3.37 (PC6)
- net GPIOC_6: now also J4.4 (Pin_4)
- net GPIOC_7: now reaches U3.38 (PC7)
- net GPIOC_7: now also J4.3 (Pin_3)
- net I2C3_SDA: now reaches U3.40 (PC9)
- net I2C3_SDA: now also J4.6 (Pin_6), R16.2
- net I2C3_SCL: now reaches U3.41 (PA8)
- net I2C3_SCL: now also J4.7 (Pin_7), R15.1
- net SPI3_NSS: now reaches U3.50 (PA15)
- net SPI3_NSS: now also J4.9 (Pin_9)
- net UART5_TX: now reaches U3.53 (PC12)
- net UART5_TX: now also J4.15 (Pin_15)
- net UART5_RX: now reaches U3.54 (PD2)
- net UART5_RX: now also J4.14 (Pin_14)
- net SPI3_SCK: now reaches U3.55 (PB3)
- net SPI3_SCK: now also J4.12 (Pin_12)
- net SPI3_MISO: now reaches U3.56 (PB4)
- net SPI3_MISO: now also J4.11 (Pin_11)
- net SPI3_MOSI: now reaches U3.57 (PB5)
- net SPI3_MOSI: now also J4.10 (Pin_10)
- no-connect marks 4 -> 17
Other:
- note added: "I2C-sensors"
- note added: "SPI-sensor"
- moved on the sheet: J1
